File: IEEEArcade/buck_converter.kicad_sch (KiCad schematic)
At the start: 3 parts, among them U4 TPS54202DDC

Commit message: Top 10 Buck Converters (Not Clickbait)
Parts:
- removed C1: 10uF, Capacitor_SMD:C_1206_3216Metric_Pad1.33x1.80mm_HandSolder, symbol Device:C
- removed R1: R, Package_TO_SOT_SMD:SOT-23-6, symbol Device:R
- added Cboot, Cin, Co: C, symbol Device:C
- added Lo: L, symbol Device:L
- added Rfb1, Rfb2: R, symbol Device:R
Connections:
- net GND: now reaches U4.1 (GND)
- net GND: now also Cin.2, Co.2, Rfb2.2
- net at U4.2 (SW): now also Cboot.2, Lo.1
- net Vin: now reaches U4.3 (VIN)
- net Vin: now also Cin.1
- net at U4.4 (FB): now also Rfb1.2, Rfb2.1
- net EN: now reaches U4.5 (EN)
- net at U4.6 (BOOT): now also Cboot.1
- new net VOUT: Co.1, Lo.2, Rfb1.1
